File: Simulation/AC-Coupled-Supply/Simulated02.sch (EAGLE design)
At the start: 3 parts

Commit message: updated to 9.5.2
Parts:
- added D1: DIODE, ngspice-simulation:DIODE
- added R2: 100k, ngspice-simulation:R
Connections:
- new net OUT: D1.C, R2.2
- net 0: now also R2.1
- net VCAP1: now also D1.A
Changed lines of the file:
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@@
 <?xml version="1.0" encoding="utf-8"?>
 <!DOCTYPE eagle SYSTEM "eagle.dtd">
-<eagle version="9.3.2">
+<eagle version="9.5.2">
 <drawing>
 <settings>
@@
 <part name="V4" library="ngspice-simulation" library_urn="urn:adsk.eagle:library:5272020" deviceset="GND" device=""/>
 <part name="V1" library="ngspice-simulation" library_urn="urn:adsk.eagle:library:5272020" deviceset="VOLTAGE" device="" value="DC 0V AC 240V"/>
+<part name="D1" library="ngspice-simulation" library_urn="urn:adsk.eagle:library:527439" deviceset="DIODE" device=""/>
+<part name="R2" library="ngspice-simulation" library_urn="urn:adsk.eagle:library:5272020" deviceset="R" device="" value="100k"/>
 </parts>
 <sheets>
@@
 <attribute name="VALUE" x="15.24" y="25.4" size="1.778" layer="96"/>
 </instance>
+<instance part="D1" gate="G$1" x="68.58" y="40.64" smashed="yes">
+<attribute name="NAME" x="63.5" y="44.45" size="1.778" layer="95"/>
+<attribute name="VALUE" x="63.5" y="30.48" size="1.778" layer="96"/>
+</instance>
+<instance part="R2" gate="G$1" x="86.36" y="25.4" smashed="yes" rot="R90">
+<attribute name="NAME" x="83.82" y="22.86" size="1.778" layer="95" rot="R90"/>
+<attribute name="VALUE" x="90.17" y="22.86" size="1.778" layer="96" rot="R90"/>
+</instance>
 </instances>
 <busses>
@@
 <label x="40.64" y="40.64" size="1.778" layer="95"/>
 <wire x1="35.56" y1="40.64" x2="43.18" y2="40.64" width="0.1524" layer="91"/>
-<wire x1="50.8" y1="40.64" x2="43.18" y2="40.64" width="0.1524" layer="91"/>
 <junction x="43.18" y="40.64"/>
 <pinref part="R1" gate="G$1" pin="2"/>
@@
 <probe x="40.64" y="50.8" size="1.778" layer="89" probetype="0"/>
 <probe x="40.64" y="48.26" size="1.778" layer="89" probetype="1"/>
-<probe x="60.96" y="45.72" size="1.778" layer="89" probetype="0"/>
+<probe x="55.88" y="53.34" size="1.778" layer="89" probetype="0"/>
+<pinref part="D1" gate="G$1" pin="A"/>
+<wire x1="43.18" y1="40.64" x2="63.5" y2="40.64" width="0.1524" layer="91"/>
 </segment>
 </net>
@@
 <pinref part="V4" gate="G$1" pin="0"/>
 <pinref part="V1" gate="G$1" pin="-"/>
+<pinref part="R2" gate="G$1" pin="1"/>
+<wire x1="43.18" y1="12.7" x2="86.36" y2="12.7" width="0.1524" layer="91"/>
+<wire x1="86.36" y1="12.7" x2="86.36" y2="20.32" width="0.1524" layer="91"/>
 </segment>
 </net>
@@
 </segment>
 </net>
+<net name="OUT" class="0">
+<segment>
+<pinref part="R2" gate="G$1" pin="2"/>
+<wire x1="86.36" y1="30.48" x2="86.36" y2="40.64" width="0.1524" layer="91"/>
+<pinref part="D1" gate="G$1" pin="C"/>
+<wire x1="86.36" y1="40.64" x2="73.66" y2="40.64" width="0.1524" layer="91"/>
+<probe x="91.44" y="48.26" size="1.778" layer="89" probetype="0"/>
+</segment>
+</net>
