File: Simulation/AC-Coupled-Supply/Simulated04.sch (EAGLE design)
At the start: 16 parts

Commit message: Simulated04.sch with linear voltage regulator 78L05
Parts:
- added C4: 100n, ngspice-simulation:C
- added IC1: 78L05Z, linear:78L05Z
- added R4: 1k, ngspice-simulation:R
- C1: value 1u -> .39u
- R2: value 120 -> 220
- R3: value 1k -> 100k
Connections:
- removed net N$5: I_LOAD.-, R3.2
- new net VOUT: IC1.VI, I_LOAD.-, R3.2
- new net V_LIN: C4.1, IC1.VO, R4.2
- net 0: now also C4.2, IC1.GND, R4.1
Other:
- moved on the sheet: R3
Changed lines of the file:
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@@
 <layers>
 <layer number="1" name="Top" color="4" fill="1" visible="no" active="no"/>
+<layer number="2" name="Route2" color="1" fill="3" visible="no" active="no"/>
+<layer number="3" name="Route3" color="4" fill="3" visible="no" active="no"/>
+<layer number="4" name="Route4" color="1" fill="4" visible="no" active="no"/>
+<layer number="5" name="Route5" color="4" fill="4" visible="no" active="no"/>
+<layer number="6" name="Route6" color="1" fill="8" visible="no" active="no"/>
+<layer number="7" name="Route7" color="4" fill="8" visible="no" active="no"/>
+<layer number="8" name="Route8" color="1" fill="2" visible="no" active="no"/>
+<layer number="9" name="Route9" color="4" fill="2" visible="no" active="no"/>
+<layer number="10" name="Route10" color="1" fill="7" visible="no" active="no"/>
+<layer number="11" name="Route11" color="4" fill="7" visible="no" active="no"/>
+<layer number="12" name="Route12" color="1" fill="5" visible="no" active="no"/>
+<layer number="13" name="Route13" color="4" fill="5" visible="no" active="no"/>
+<layer number="14" name="Route14" color="1" fill="6" visible="no" active="no"/>
+<layer number="15" name="Route15" color="4" fill="6" visible="no" active="no"/>
 <layer number="16" name="Bottom" color="1" fill="1" visible="no" active="no"/>
 <layer number="17" name="Pads" color="2" fill="1" visible="no" active="no"/>
@@
 </part>
 <part name="X_3" library="ngspice-simulation" library_urn="urn:adsk.eagle:library:5272020" deviceset="GND" device=""/>
-<part name="R2" library="ngspice-simulation" library_urn="urn:adsk.eagle:library:5272020" deviceset="R" device="" value="120"/>
-<part name="C1" library="ngspice-simulation" library_urn="urn:adsk.eagle:library:527439" deviceset="C" device="" value="1u"/>
+<part name="R2" library="ngspice-simulation" library_urn="urn:adsk.eagle:library:5272020" deviceset="R" device="" value="220"/>
+<part name="C1" library="ngspice-simulation" library_urn="urn:adsk.eagle:library:527439" deviceset="C" device="" value=".39u"/>
 <part name="D5" library="ngspice-simulation" library_urn="urn:adsk.eagle:library:527439" deviceset="DIODE" device="" value="">
 <spice>
@@
 </part>
 <part name="VCUR_2" library="ngspice-simulation" library_urn="urn:adsk.eagle:library:527439" deviceset="AMMETER" device=""/>
-<part name="R3" library="ngspice-simulation" library_urn="urn:adsk.eagle:library:5272020" deviceset="R" device="" value="1k"/>
+<part name="R3" library="ngspice-simulation" library_urn="urn:adsk.eagle:library:5272020" deviceset="R" device="" value="100k"/>
 <part name="C3" library="ngspice-simulation" library_urn="urn:adsk.eagle:library:527439" deviceset="C" device="" value="47u"/>
 <part name="I_LOAD" library="ngspice-simulation" library_urn="urn:adsk.eagle:library:527439" deviceset="AMMETER" device=""/>
+<part name="IC1" library="linear" library_urn="urn:adsk.eagle:library:262" deviceset="78*" device="Z" package3d_urn="urn:adsk.eagle:package:16416/2" technology="L05">
+<spice>
+<pinmapping isusermap="yes" isdevicewide="no">
+<pinmap gate="A1" pin="GND" pinorder="2"/>
+<pinmap gate="A1" pin="VI" pinorder="1"/>
+<pinmap gate="A1" pin="VO" pinorder="3"/>
+</pinmapping>
+</spice>
+<attribute name="SPICEMODEL" value="LM7805"/>
+<attribute name="SPICEPREFIX" value="X"/>
+</part>
+<part name="C4" library="ngspice-simulation" library_urn="urn:adsk.eagle:library:527439" deviceset="C" device="" value="100n"/>
+<part name="R4" library="ngspice-simulation" library_urn="urn:adsk.eagle:library:5272020" deviceset="R" device="" value="1k"/>
 </parts>
 <sheets>
@@
 <attribute name="NAME" x="180.34" y="35.56" size="1.778" layer="95" rot="R90"/>
 </instance>
-<instance part="R3" gate="G$1" x="246.38" y="12.7" smashed="yes" rot="R90">
-<attribute name="NAME" x="243.84" y="10.16" size="1.778" layer="95" rot="R90"/>
-<attribute name="VALUE" x="250.19" y="10.16" size="1.778" layer="96" rot="R90"/>
+<instance part="R3" gate="G$1" x="246.38" y="10.16" smashed="yes" rot="R90">
+<attribute name="NAME" x="243.84" y="7.62" size="1.778" layer="95" rot="R90"/>
+<attribute name="VALUE" x="250.19" y="7.62" size="1.778" layer="96" rot="R90"/>
 </instance>
 <instance part="C3" gate="G$1" x="210.82" y="12.7" smashed="yes">
@@
 <instance part="I_LOAD" gate="G$1" x="231.14" y="25.4" smashed="yes" rot="R90">
 <attribute name="NAME" x="236.22" y="33.02" size="1.778" layer="95" rot="R180"/>
+</instance>
+<instance part="IC1" gate="A1" x="274.32" y="25.4" smashed="yes">
+<attribute name="NAME" x="266.7" y="31.115" size="1.778" layer="95"/>
+<attribute name="VALUE" x="266.7" y="28.575" size="1.778" layer="96"/>
+</instance>
+<instance part="C4" gate="G$1" x="292.1" y="10.16" smashed="yes">
+<attribute name="NAME" x="294.64" y="12.7" size="1.778" layer="95"/>
+<attribute name="VALUE" x="294.64" y="10.16" size="1.778" layer="96"/>
+</instance>
+<instance part="R4" gate="G$1" x="309.88" y="10.16" smashed="yes" rot="R90">
+<attribute name="NAME" x="307.34" y="7.62" size="1.778" layer="95" rot="R90"/>
+<attribute name="VALUE" x="313.69" y="7.62" size="1.778" layer="96" rot="R90"/>
 </instance>
 </instances>
@@
 <pinref part="R3" gate="G$1" pin="1"/>
 <wire x1="210.82" y1="-2.54" x2="246.38" y2="-2.54" width="0.1524" layer="91"/>
-<wire x1="246.38" y1="-2.54" x2="248.92" y2="-2.54" width="0.1524" layer="91"/>
-<wire x1="246.38" y1="7.62" x2="246.38" y2="-2.54" width="0.1524" layer="91"/>
+<wire x1="246.38" y1="5.08" x2="246.38" y2="-2.54" width="0.1524" layer="91"/>
 <junction x="246.38" y="-2.54"/>
 <pinref part="C3" gate="G$1" pin="2"/>
 <wire x1="210.82" y1="7.62" x2="210.82" y2="-2.54" width="0.1524" layer="91"/>
 <junction x="210.82" y="-2.54"/>
+<pinref part="IC1" gate="A1" pin="GND"/>
+<wire x1="274.32" y1="17.78" x2="274.32" y2="-2.54" width="0.1524" layer="91"/>
+<wire x1="274.32" y1="-2.54" x2="246.38" y2="-2.54" width="0.1524" layer="91"/>
+<wire x1="274.32" y1="-2.54" x2="292.1" y2="-2.54" width="0.1524" layer="91"/>
+<junction x="274.32" y="-2.54"/>
+<pinref part="R4" gate="G$1" pin="1"/>
+<wire x1="292.1" y1="-2.54" x2="309.88" y2="-2.54" width="0.1524" layer="91"/>
+<wire x1="309.88" y1="-2.54" x2="309.88" y2="5.08" width="0.1524" layer="91"/>
+<pinref part="C4" gate="G$1" pin="2"/>
+<wire x1="292.1" y1="5.08" x2="292.1" y2="-2.54" width="0.1524" layer="91"/>
+<junction x="292.1" y="-2.54"/>
 </segment>
 </net>
@@
 <wire x1="200.66" y1="25.4" x2="193.04" y2="25.4" width="0.1524" layer="91"/>
 <pinref part="D6" gate="G$1" pin="C"/>
-<probe x="200.66" y="27.94" size="1.778" layer="89" probetype="0"/>
 <wire x1="200.66" y1="25.4" x2="210.82" y2="25.4" width="0.1524" layer="91"/>
 <junction x="200.66" y="25.4"/>
@@
 </segment>
 </net>
-<net name="N$5" class="0">
+<net name="VOUT" class="0">
 <segment>
 <pinref part="R3" gate="G$1" pin="2"/>
-<wire x1="246.38" y1="25.4" x2="246.38" y2="17.78" width="0.1524" layer="91"/>
+<wire x1="246.38" y1="25.4" x2="246.38" y2="15.24" width="0.1524" layer="91"/>
 <wire x1="238.76" y1="25.4" x2="246.38" y2="25.4" width="0.1524" layer="91"/>
 <pinref part="I_LOAD" gate="G$1" pin="-"/>
+<probe x="246.38" y="38.1" size="1.778" layer="89" rot="R180" probetype="0"/>
+<pinref part="IC1" gate="A1" pin="VI"/>
+<wire x1="264.16" y1="25.4" x2="246.38" y2="25.4" width="0.1524" layer="91"/>
+<junction x="246.38" y="25.4"/>
+</segment>
+</net>
+<net name="V_LIN" class="0">
+<segment>
+<pinref part="IC1" gate="A1" pin="VO"/>
+<wire x1="284.48" y1="25.4" x2="292.1" y2="25.4" width="0.1524" layer="91"/>
+<probe x="299.72" y="33.02" size="1.778" layer="89" probetype="0"/>
+<pinref part="R4" gate="G$1" pin="2"/>
+<wire x1="292.1" y1="25.4" x2="309.88" y2="25.4" width="0.1524" layer="91"/>
+<wire x1="309.88" y1="15.24" x2="309.88" y2="25.4" width="0.1524" layer="91"/>
+<pinref part="C4" gate="G$1" pin="1"/>
+<wire x1="292.1" y1="12.7" x2="292.1" y2="25.4" width="0.1524" layer="91"/>
+<junction x="292.1" y="25.4"/>
 </segment>
 </net>
@@
 will not be understood (or retained) with this version.
 </note>
+<note version="8.3" severity="warning">
+Since Version 8.3, EAGLE supports the association of 3D packages
+with devices in libraries, schematics, and board files. Those 3D
+packages will not be understood (or retained) with this version.
+</note>
 <note version="8.4" severity="warning">
